File: manufacturing/PCB/Shield/shield.sch (EAGLE design)
At the start: 230 parts, among them J1 DC_JACK, Q1 12 MHz, T1 PHKD3NQ10T, U1 UCC27531, U10 UCC27531, U11 UCC27531, U12 UCC27531, U13 UCC27531, U14 UCC27531, U15 UCC27531, U16 UCC27531, U17 UCC27531, U18 UCC27531, U19 UCC27531, U2 UCC27531, U20 UCC27531, U21 UCC27531, U22 UCC27531, U23 UCC27531, U24 UCC27531, U25 UCC27531, U26 UCC27531, U27 UCC27531, U28 UCC27531, U29 UCC27531, U3 UCC27531, U30 UCC27531, U31 UCC27531, U32 UCC27531, U33 UCC27531, U34 UCC27531, U35 UCC27531, U36 UCC27531, U37 UCC27531, U38 UCC27531, U39 UCC27531, U4 UCC27531, U40 UCC27531, U41 UCC27531, U42 UCC27531, U43 UCC27531, U44 UCC27531, U45 UCC27531, U46 UCC27531, U47 UCC27531, U48 UCC27531, U49 UCC27531, U5 UCC27531, U50 UCC27531, U51 UCC27531, U52 UCC27531, U53 UCC27531, U54 UCC27531, U55 UCC27531, U56 UCC27531, U57 UCC27531, U58 UCC27531, U59 UCC27531, U6 UCC27531, U60 UCC27531, U61 UCC27531, U62 UCC27531, U63 UCC27531, U64 UCC27531, U65 LTC4365, U66 FT232R, U7 UCC27531, U8 UCC27531, U9 UCC27531, X1 MINI-USB, X2 BNC

Commit message: fixed RX/TX swap, added power from USB option (Shield v1.1 ready for production)
Parts:
- removed C1: 1uF, eagle-ltspice:C
- added R8: 0R, rcl:R-EU_R0805
Connections:
- new net N$1: JP1.12, R8.2
- net GND: no longer C1.2
- net RX: now also JP1.1; no longer JP1.2
- net TX: now also JP1.2; no longer JP1.1
- net VBUS: now also R8.1
- net VDD: no longer C1.1
